File: ps/ps.brd (EAGLE design)
At the start: 99.1 x 54.6 mm, 66 parts, among them IC1 LM675, Q1 NPN-D, Q2 NPN-D, U1 LM3480IM4, U2 LM317, U3 TLC555CD, U4 LM317, U5 LM317

Commit message: Some tweaks
Parts:
- added R15: 6.8/0.5W, SparkFun-Resistors:AXIAL-0.5
- R10: value 3.4/1W -> 6.8/0.5W; device SparkFun-Resistors:AXIAL-0.6 -> SparkFun-Resistors:AXIAL-0.5
- moved R10 2.29 mm to (10.2, 46.4)
Connections:
- net H+: now also R15.P$2
- net N$8: now also R15.P$1
Routing:
- net VINF: track 125.9 -> 116.5 mm, vias 8 -> 5
- net H+: track 62.7 -> 67.7 mm
- net N$8: track 8.98 -> 9.83 mm
Changed lines of the file:
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@@
 <attribute name="NAME" x="43.18" y="0.762" size="0.8128" layer="25" ratio="15"/>
 </element>
-<element name="R10" library="SparkFun-Resistors" package="AXIAL-0.6" value="3.4/1W" x="11.43" y="44.45" smashed="yes" rot="R180">
-<attribute name="NAME" x="8.255" y="41.91" size="0.8128" layer="25" font="vector" ratio="15" rot="R180"/>
-<attribute name="VALUE" x="15.494" y="44.831" size="0.8128" layer="21" font="vector" ratio="15" rot="R180"/>
+<element name="R10" library="SparkFun-Resistors" package="AXIAL-0.5" value="6.8/0.5W" x="10.16" y="46.355" smashed="yes" rot="R180">
+<attribute name="NAME" x="17.78" y="45.085" size="0.8128" layer="25" font="vector" ratio="15" rot="R180"/>
+<attribute name="VALUE" x="12.954" y="46.736" size="0.8128" layer="21" font="vector" ratio="15" rot="R180"/>
 </element>
 <element name="U4" library="my" package="TO220BV" value="LM317" x="12.7" y="53.34" smashed="yes">
 <attribute name="NAME" x="6.35" y="49.1998" size="0.8128" layer="25" ratio="15"/>
-<attribute name="VALUE" x="6.35" y="47.625" size="0.8128" layer="27" ratio="15"/>
+<attribute name="VALUE" x="15.875" y="47.625" size="0.8128" layer="27" ratio="15"/>
 </element>
 <element name="J1" library="SparkFun-Connectors" package="1X02" value="" x="83.82" y="27.94" smashed="yes" rot="R90">
@@
 <attribute name="VALUE" x="79.121" y="29.718" size="0.8128" layer="27" font="vector" ratio="15" rot="R180"/>
 </element>
+<element name="R15" library="SparkFun-Resistors" package="AXIAL-0.5" value="6.8/0.5W" x="10.16" y="42.545" rot="R180"/>
 </elements>
 <signals>
@@
 <wire x1="53.645" y1="49.225" x2="53.645" y2="46.99" width="0.6096" layer="1"/>
 <wire x1="52.07" y1="50.8" x2="38.1" y2="36.83" width="1.27" layer="16" curve="-90"/>
-<wire x1="38.1" y1="36.83" x2="16.51" y2="36.83" width="1.27" layer="16"/>
-<wire x1="12.7" y1="31.75" x2="12.7" y2="36.83" width="1.27" layer="1"/>
-<via x="12.7" y="43.18" extent="1-16" drill="0.6"/>
-<wire x1="12.7" y1="36.83" x2="12.7" y2="40.64" width="1.27" layer="1"/>
-<wire x1="12.7" y1="40.64" x2="12.7" y2="41.91" width="1.27" layer="1"/>
-<wire x1="12.7" y1="41.91" x2="12.7" y2="43.18" width="1.27" layer="1"/>
-<wire x1="19.44" y1="41.91" x2="12.7" y2="41.91" width="1.27" layer="1"/>
+<wire x1="38.1" y1="36.83" x2="17.78" y2="36.83" width="1.27" layer="16"/>
+<wire x1="17.78" y1="36.83" x2="16.51" y2="36.83" width="1.27" layer="1"/>
 <wire x1="16.51" y1="36.83" x2="15.24" y2="36.83" width="1.27" layer="1"/>
-<wire x1="15.24" y1="36.83" x2="13.97" y2="36.83" width="1.27" layer="1"/>
-<wire x1="13.97" y1="36.83" x2="12.7" y2="36.83" width="1.27" layer="1"/>
-<via x="13.97" y="36.83" extent="1-16" drill="0.6"/>
+<via x="15.24" y="36.83" extent="1-16" drill="0.6"/>
+<wire x1="17.78" y1="36.83" x2="16.51" y2="36.83" width="1.27" layer="16"/>
 <wire x1="16.51" y1="36.83" x2="15.24" y2="36.83" width="1.27" layer="16"/>
-<wire x1="15.24" y1="36.83" x2="13.97" y2="36.83" width="1.27" layer="16"/>
-<via x="15.24" y="36.83" extent="1-16" drill="0.6"/>
 <via x="16.51" y="36.83" extent="1-16" drill="0.6"/>
-<via x="12.7" y="40.64" extent="1-16" drill="0.6"/>
-<wire x1="12.7" y1="40.64" x2="12.7" y2="41.91" width="1.27" layer="16"/>
-<wire x1="12.7" y1="41.91" x2="12.7" y2="43.18" width="1.27" layer="16"/>
-<wire x1="12.7" y1="43.18" x2="13.97" y2="44.45" width="1.27" layer="16" curve="-90"/>
-<wire x1="13.97" y1="44.45" x2="15.24" y2="45.72" width="1.27" layer="16" curve="90"/>
-<wire x1="15.24" y1="45.72" x2="15.24" y2="50.8" width="1.27" layer="16"/>
-<via x="12.7" y="41.91" extent="1-16" drill="0.6"/>
+<via x="17.78" y="36.83" extent="1-16" drill="0.6"/>
+<wire x1="17.78" y1="36.83" x2="17.78" y2="40.25" width="1.27" layer="1"/>
+<wire x1="17.78" y1="40.25" x2="19.44" y2="41.91" width="1.27" layer="1" curve="-90"/>
+<wire x1="12.7" y1="31.75" x2="12.7" y2="34.29" width="1.27" layer="1"/>
+<wire x1="12.7" y1="34.29" x2="15.24" y2="36.83" width="1.27" layer="1" curve="-90"/>
+<wire x1="19.44" y1="41.91" x2="19.44" y2="46.6" width="1.27" layer="1"/>
+<wire x1="19.44" y1="46.6" x2="15.24" y2="50.8" width="1.27" layer="1" curve="90"/>
 </signal>
 <signal name="VREG" class="1">
@@
 <contactref element="U4" pad="1"/>
 <contactref element="R10" pad="P$2"/>
-<wire x1="3.81" y1="44.45" x2="10.16" y2="50.8" width="0.6096" layer="1" curve="90"/>
 <wire x1="34.29" y1="4.445" x2="32.385" y2="4.445" width="0.6096" layer="16"/>
 <wire x1="32.385" y1="4.445" x2="7.62" y2="29.21" width="0.6096" layer="16" curve="-90"/>
-<wire x1="7.62" y1="29.21" x2="7.62" y2="40.64" width="0.6096" layer="16"/>
-<wire x1="7.62" y1="40.64" x2="3.81" y2="44.45" width="0.6096" layer="16" curve="90"/>
+<contactref element="R15" pad="P$2"/>
+<wire x1="7.62" y1="29.21" x2="7.62" y2="41.91" width="0.6096" layer="16"/>
+<wire x1="7.62" y1="41.91" x2="7.62" y2="46.99" width="0.6096" layer="16"/>
+<wire x1="7.62" y1="46.99" x2="7.62" y2="48.26" width="0.6096" layer="16"/>
+<wire x1="7.62" y1="48.26" x2="10.16" y2="50.8" width="0.6096" layer="16" curve="-90"/>
+<wire x1="3.81" y1="42.545" x2="6.985" y2="42.545" width="0.6096" layer="16"/>
+<wire x1="6.985" y1="42.545" x2="7.62" y2="41.91" width="0.6096" layer="16" curve="-90"/>
+<wire x1="3.81" y1="46.355" x2="6.985" y2="46.355" width="0.6096" layer="16"/>
+<wire x1="6.985" y1="46.355" x2="7.62" y2="46.99" width="0.6096" layer="16" curve="90"/>
 </signal>
 <signal name="N$8">
 <contactref element="U4" pad="2"/>
 <contactref element="R10" pad="P$1"/>
-<wire x1="19.05" y1="44.45" x2="12.7" y2="50.8" width="0.6096" layer="1" curve="-90"/>
+<contactref element="R15" pad="P$1"/>
+<wire x1="16.51" y1="42.545" x2="16.51" y2="46.355" width="0.6096" layer="1"/>
+<wire x1="12.7" y1="50.8" x2="12.7" y2="50.165" width="0.6096" layer="1"/>
+<wire x1="12.7" y1="50.165" x2="16.51" y2="46.355" width="0.6096" layer="1" curve="90"/>
 </signal>
 <signal name="N$5">

Commit message: PSU tweaked
Parts:
- R5: value 4.7K -> 1K/0.5W; device SparkFun-Resistors:0603-RES -> rcl:R1210W
- moved C1 0.63 mm to (24.8, 17.8)
Routing:
- net VINF: track 116.5 -> 119.9 mm
Changed lines of the file:
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@@
 <attribute name="VALUE" x="57.315" y="20.06" size="1.016" layer="27" ratio="15" rot="R90"/>
 </element>
-<element name="C1" library="SparkFun-Capacitors" package="0603-CAP" value="0.1uF" x="25.4" y="17.78" smashed="yes" rot="R90">
-<attribute name="PROD_ID" value="CAP-00810" x="25.4" y="17.78" size="1.778" layer="27" rot="R90" display="off"/>
-<attribute name="NAME" x="25.654" y="20.193" size="0.8128" layer="25" font="vector" ratio="15" rot="R180"/>
-<attribute name="VALUE" x="25.781" y="15.748" size="0.8128" layer="27" font="vector" ratio="15" rot="R180"/>
+<element name="C1" library="SparkFun-Capacitors" package="0603-CAP" value="0.1uF" x="24.765" y="17.78" smashed="yes" rot="R90">
+<attribute name="PROD_ID" value="CAP-00810" x="24.765" y="17.78" size="1.778" layer="27" rot="R90" display="off"/>
+<attribute name="NAME" x="25.019" y="20.193" size="0.8128" layer="25" font="vector" ratio="15" rot="R180"/>
+<attribute name="VALUE" x="25.146" y="15.748" size="0.8128" layer="27" font="vector" ratio="15" rot="R180"/>
 </element>
 <element name="C5" library="SparkFun-Capacitors" package="0603-CAP" value="10nF" x="34.29" y="19.05" smashed="yes">
@@
 <attribute name="VALUE" x="42.926" y="13.208" size="0.8128" layer="27" font="vector" ratio="15" rot="R180"/>
 </element>
-<element name="R5" library="SparkFun-Resistors" package="0603-RES" value="4.7K" x="29.21" y="19.05" smashed="yes" rot="R180">
-<attribute name="PROD_ID" value="RES-07857" x="29.21" y="19.05" size="1.778" layer="27" rot="R180" display="off"/>
-<attribute name="NAME" x="30.099" y="18.288" size="0.8128" layer="25" font="vector" ratio="15" rot="R180"/>
-<attribute name="VALUE" x="30.861" y="20.828" size="0.8128" layer="27" font="vector" ratio="15" rot="R180"/>
+<element name="R5" library="rcl" package="R1210W" value="1K/0.5W" x="29.21" y="19.05" smashed="yes" rot="R180">
+<attribute name="NAME" x="30.099" y="17.653" size="0.8128" layer="25" font="vector" ratio="15" rot="R180"/>
 </element>
 <element name="R11" library="SparkFun-Resistors" package="AXIAL-0.4" value="56.2K" x="76.2" y="21.59" smashed="yes" rot="R270">
@@
 <wire x1="35.391" y1="21.98" x2="37.541" y2="24.13" width="1.27" layer="1" curve="90"/>
 <wire x1="37.541" y1="24.13" x2="43.7388" y2="24.13" width="1.27" layer="1"/>
-<wire x1="30.06" y1="19.05" x2="30.48" y2="19.47" width="1.27" layer="1" curve="90"/>
+<wire x1="30.709" y1="19.05" x2="30.48" y2="19.47" width="1.27" layer="1" curve="90"/>
 <wire x1="30.48" y1="19.47" x2="30.48" y2="21.8186" width="1.27" layer="1"/>
 </signal>
@@
 <contactref element="Q2" pad="4"/>
 <contactref element="R5" pad="2"/>
-<wire x1="28.4988" y1="24.13" x2="27.94" y2="24.13" width="1.27" layer="1"/>
-<wire x1="27.94" y1="24.13" x2="22.301" y2="24.13" width="1.27" layer="1"/>
-<wire x1="26.99" y1="14.97" x2="25.4" y2="16.56" width="0.4064" layer="1" curve="-90"/>
-<wire x1="25.4" y1="16.56" x2="25.4" y2="16.93" width="0.4064" layer="1"/>
-<wire x1="25.4" y1="16.93" x2="26.24" y2="16.93" width="0.4064" layer="1"/>
-<wire x1="26.24" y1="16.93" x2="28.36" y2="19.05" width="0.4064" layer="1" curve="90"/>
-<wire x1="28.36" y1="19.05" x2="27.94" y2="19.05" width="0.4064" layer="1"/>
-<via x="27.94" y="19.05" extent="1-16" drill="0.6"/>
-<wire x1="27.94" y1="19.05" x2="27.94" y2="24.13" width="0.4064" layer="16"/>
-<via x="27.94" y="24.13" extent="1-16" drill="0.6"/>
+<wire x1="28.4988" y1="24.13" x2="29.21" y2="24.13" width="1.27" layer="1"/>
+<wire x1="29.21" y1="24.13" x2="22.301" y2="24.13" width="1.27" layer="1"/>
+<wire x1="27.711" y1="19.05" x2="27.94" y2="19.05" width="0.4064" layer="1"/>
+<via x="29.21" y="24.13" extent="1-16" drill="0.6"/>
 <contactref element="U4" pad="3"/>
 <wire x1="6.35" y1="20.53" x2="12.7" y2="26.88" width="1.27" layer="1" curve="90"/>
@@
 <wire x1="19.44" y1="41.91" x2="19.44" y2="46.6" width="1.27" layer="1"/>
 <wire x1="19.44" y1="46.6" x2="15.24" y2="50.8" width="1.27" layer="1" curve="90"/>
+<wire x1="27.94" y1="19.05" x2="26.67" y2="19.05" width="0.6096" layer="1"/>
+<via x="26.67" y="19.05" extent="1-16" drill="0.6"/>
+<wire x1="26.67" y1="19.05" x2="26.67" y2="21.59" width="0.6096" layer="16"/>
+<wire x1="26.67" y1="21.59" x2="29.21" y2="24.13" width="0.6096" layer="16" curve="-90"/>
+<wire x1="26.99" y1="14.97" x2="26.67" y2="15.29" width="0.6096" layer="1" curve="-90"/>
+<wire x1="26.67" y1="15.29" x2="26.67" y2="16.51" width="0.6096" layer="1"/>
+<wire x1="26.67" y1="16.51" x2="26.67" y2="19.05" width="0.6096" layer="1"/>
+<wire x1="24.765" y1="16.93" x2="25.185" y2="16.51" width="0.6096" layer="1" curve="90"/>
+<wire x1="25.185" y1="16.51" x2="26.67" y2="16.51" width="0.6096" layer="1"/>
 </signal>
 <signal name="VREG" class="1">

Commit message: PSU tweaked
Parts:
- R2: value 10K -> 4.7K
- U1: value LM3480IM4 -> (none); device my:SOT23-3 -> my:SOT-89
Connections:
- net GND: now also U1.2, U1.PAD; no longer U1.3
- net VINF: now also U1.3; no longer U1.2
Routing:
- net VINF: track 119.9 -> 119.0 mm
Changed lines of the file:
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@@
 <attribute name="VALUE" x="40.8305" y="23.0505" size="0.8128" layer="27" ratio="15" rot="R90"/>
 </element>
-<element name="R2" library="SparkFun-Resistors" package="0603-RES" value="10K" x="45.72" y="19.05" smashed="yes">
+<element name="R2" library="SparkFun-Resistors" package="0603-RES" value="4.7K" x="45.72" y="19.05" smashed="yes">
 <attribute name="PROD_ID" value="RES-00824" x="45.72" y="19.05" size="1.778" layer="27" display="off"/>
 <attribute name="NAME" x="44.831" y="19.812" size="0.8128" layer="25" font="vector" ratio="15"/>
@@
 <attribute name="VALUE" x="37.4396" y="18.2626" size="0.8128" layer="27" ratio="15" rot="SR0"/>
 </element>
-<element name="U1" library="my" package="SOT23-3" value="LM3480IM4" x="27.94" y="13.97" smashed="yes" rot="R180">
-<attribute name="NAME" x="26.2255" y="14.097" size="0.8128" layer="25" ratio="15" rot="R180"/>
+<element name="U1" library="my" package="SOT-89" value="" x="27.94" y="13.97" smashed="yes" rot="R180">
+<attribute name="NAME" x="24.9555" y="14.097" size="0.8128" layer="25" ratio="15" rot="R180"/>
 <attribute name="VALUE" x="26.416" y="12.8905" size="0.8128" layer="27" ratio="15" rot="R180"/>
 </element>
@@
 <wire x1="36.83" y1="17.78" x2="38.6588" y2="17.78" width="0.4064" layer="1"/>
 <wire x1="38.6588" y1="17.78" x2="39.2938" y2="17.145" width="0.4064" layer="1" curve="-90"/>
-<wire x1="28.89" y1="14.97" x2="29.52" y2="14.34" width="0.4064" layer="1" curve="90"/>
-<wire x1="29.52" y1="14.34" x2="31.75" y2="14.34" width="0.4064" layer="1"/>
 <wire x1="31.75" y1="14.34" x2="32.755" y2="13.335" width="0.4064" layer="1" curve="90"/>
 <wire x1="32.755" y1="13.335" x2="34.3662" y2="13.335" width="0.4064" layer="1"/>
+<wire x1="31.75" y1="14.34" x2="30.999" y2="14.34" width="0.6096" layer="1"/>
+<wire x1="30.999" y1="14.34" x2="29.464" y2="15.875" width="0.6096" layer="1" curve="-90"/>
 </signal>
 <signal name="GND">
 <contactref element="C1" pad="2"/>
-<contactref element="U1" pad="3"/>
+<contactref element="U1" pad="2"/>
 <contactref element="C3" pad="2"/>
 <contactref element="U3" pad="1"/>
@@
 <via x="73.66" y="31.75" extent="1-16" drill="0.6"/>
 <via x="80.01" y="34.29" extent="1-16" drill="0.6"/>
+<contactref element="U1" pad="PAD"/>
 </signal>
 <signal name="555CONT">
@@
 <contactref element="C4" pad="1"/>
 <contactref element="C1" pad="1"/>
-<contactref element="U1" pad="2"/>
+<contactref element="U1" pad="3"/>
 <contactref element="D4" pad="A"/>
 <contactref element="Q2" pad="2"/>
@@
 <wire x1="26.67" y1="19.05" x2="26.67" y2="21.59" width="0.6096" layer="16"/>
 <wire x1="26.67" y1="21.59" x2="29.21" y2="24.13" width="0.6096" layer="16" curve="-90"/>
-<wire x1="26.99" y1="14.97" x2="26.67" y2="15.29" width="0.6096" layer="1" curve="-90"/>
-<wire x1="26.67" y1="15.29" x2="26.67" y2="16.51" width="0.6096" layer="1"/>
-<wire x1="26.67" y1="16.51" x2="26.67" y2="19.05" width="0.6096" layer="1"/>
-<wire x1="24.765" y1="16.93" x2="25.185" y2="16.51" width="0.6096" layer="1" curve="90"/>
-<wire x1="25.185" y1="16.51" x2="26.67" y2="16.51" width="0.6096" layer="1"/>
+<wire x1="26.416" y1="15.875" x2="26.67" y2="16.129" width="0.6096" layer="1" curve="90"/>
+<wire x1="26.67" y1="16.129" x2="26.67" y2="19.05" width="0.6096" layer="1"/>
+<wire x1="24.765" y1="16.93" x2="25.361" y2="16.93" width="0.6096" layer="1"/>
+<wire x1="25.361" y1="16.93" x2="26.416" y2="15.875" width="0.6096" layer="1" curve="-90"/>
 </signal>
 <signal name="VREG" class="1">
