File: ps/ps.sch (EAGLE design)
At the start: 67 parts, among them IC1 LM675, Q1 NPN-D, Q2 NPN-D, U1 LM3480IM4, U2 LM317, U3 TLC555CD, U4 LM317, U5 LM317

Commit message: PSU tweaked
Parts:
- R2: value 10K -> 4.7K
- U1: value LM3480IM4 -> (none); device my:LM3480IM4 -> my:L78L12ACUTR
Changed lines of the file:
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@@
 <part name="Q1" library="my" deviceset="NPN-D" device=""/>
 <part name="U3" library="Texas Instruments_By_element14_Batch_1" deviceset="TLC555CD" device=""/>
-<part name="U1" library="my" deviceset="LM3480IM4" device=""/>
+<part name="U1" library="my" deviceset="L78L12ACUTR" device=""/>
 <part name="C3" library="SparkFun-Capacitors" deviceset="1.0UF-25V-+80/-20(0805)" device="&quot;" value="1.0uF"/>
 <part name="C1" library="SparkFun-Capacitors" deviceset="0.1UF-25V(+80/-20%)(0603)" device="" value="0.1uF"/>
@@
 <part name="C5" library="SparkFun-Capacitors" deviceset="10NF/10000PF-50V-10%(0603)" device="" value="10nF"/>
 <part name="GND7" library="SparkFun-Aesthetics" deviceset="GND" device=""/>
-<part name="R2" library="SparkFun-Resistors" deviceset="10KOHM-1/10W-1%(0603)" device="0603" value="10K"/>
+<part name="R2" library="SparkFun-Resistors" deviceset="10KOHM-1/10W-1%(0603)" device="0603" value="4.7K"/>
 <part name="C10" library="SparkFun-Capacitors" deviceset="470PF-50V-5%(0603)" device="SMD" value="470pF"/>
 <part name="GND11" library="SparkFun-Aesthetics" deviceset="GND" device=""/>
@@
 <pinref part="U1" gate="G$1" pin="OUT"/>
 <pinref part="C3" gate="G$1" pin="1"/>
-<wire x1="50.8" y1="76.2" x2="53.34" y2="76.2" width="0.1524" layer="91"/>
+<wire x1="49.53" y1="76.2" x2="53.34" y2="76.2" width="0.1524" layer="91"/>
 <wire x1="53.34" y1="76.2" x2="53.34" y2="73.66" width="0.1524" layer="91"/>
 <pinref part="U3" gate="A" pin="VDD"/>
@@
 <pinref part="U1" gate="G$1" pin="GND"/>
 <pinref part="GND4" gate="1" pin="GND"/>
+<wire x1="38.1" y1="66.04" x2="38.1" y2="68.58" width="0.1524" layer="91"/>
 </segment>
 <segment>
@@
 <wire x1="22.86" y1="73.66" x2="22.86" y2="76.2" width="0.1524" layer="91"/>
 <pinref part="U1" gate="G$1" pin="IN"/>
-<wire x1="22.86" y1="76.2" x2="25.4" y2="76.2" width="0.1524" layer="91"/>
+<wire x1="22.86" y1="76.2" x2="26.67" y2="76.2" width="0.1524" layer="91"/>
 <wire x1="22.86" y1="76.2" x2="20.32" y2="76.2" width="0.1524" layer="91"/>
 <junction x="22.86" y="76.2"/>

Commit message: More filtering
Parts:
- added R16: 0.33, rcl:R-US_R0805
- C13, C14, C15, C16, C17, C18, C21, C25: value 1u/250V -> 2.2u/250V
- C26: value 0.1uF/250V -> 1uF/100V; device rcl:C-EUC1206 -> SparkFun-Capacitors:CAP1210
- L1: value 100u -> 220u; device SparkFun-Passives:INDUCTOR-B82462G -> my:INDUCTORNR10050T-PTH-ADD
Connections:
- net VCC: now also R16.1
- net VINF: now also R16.2
Other:
- moved on the sheet: C26
Changed lines of the file:
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@@
 <part name="D11" library="SparkFun-DiscreteSemi" deviceset="DIODE-SCHOTTKY" device="-B340A" value="1A/40V"/>
 <part name="FRAME1" library="frames" deviceset="A3L-LOC" device=""/>
-<part name="C13" library="rcl" deviceset="C-EU" device="C2220K" value="1u/250V"/>
-<part name="C14" library="rcl" deviceset="C-EU" device="C2220K" value="1u/250V"/>
-<part name="C15" library="rcl" deviceset="C-EU" device="C2220K" value="1u/250V"/>
-<part name="C16" library="rcl" deviceset="C-EU" device="C2220K" value="1u/250V"/>
-<part name="C17" library="rcl" deviceset="C-EU" device="C2220K" value="1u/250V"/>
-<part name="C18" library="rcl" deviceset="C-EU" device="C2220K" value="1u/250V"/>
-<part name="C21" library="rcl" deviceset="C-EU" device="C2220K" value="1u/250V"/>
+<part name="C13" library="rcl" deviceset="C-EU" device="C2220K" value="2.2u/250V"/>
+<part name="C14" library="rcl" deviceset="C-EU" device="C2220K" value="2.2u/250V"/>
+<part name="C15" library="rcl" deviceset="C-EU" device="C2220K" value="2.2u/250V"/>
+<part name="C16" library="rcl" deviceset="C-EU" device="C2220K" value="2.2u/250V"/>
+<part name="C17" library="rcl" deviceset="C-EU" device="C2220K" value="2.2u/250V"/>
+<part name="C18" library="rcl" deviceset="C-EU" device="C2220K" value="2.2u/250V"/>
+<part name="C21" library="rcl" deviceset="C-EU" device="C2220K" value="2.2u/250V"/>
 <part name="GND12" library="SparkFun-Aesthetics" deviceset="GND" device=""/>
 <part name="GND14" library="SparkFun-Aesthetics" deviceset="GND" device=""/>
@@
 <part name="GND19" library="SparkFun-Aesthetics" deviceset="GND" device=""/>
 <part name="U5" library="SparkFun-PowerIC" deviceset="V_REG_317" device="DPACK" value="LM317"/>
-<part name="C25" library="rcl" deviceset="C-EU" device="C2220K" value="1u/250V"/>
+<part name="C25" library="rcl" deviceset="C-EU" device="C2220K" value="2.2u/250V"/>
 <part name="GND20" library="SparkFun-Aesthetics" deviceset="GND" device=""/>
 <part name="R11" library="SparkFun-Resistors" deviceset="RESISTOR" device="PTH-1/4W" value="56.2K"/>
@@
 <part name="GND22" library="SparkFun-Aesthetics" deviceset="GND" device=""/>
 <part name="R12" library="SparkFun-Resistors" deviceset="RESISTOR" device="PTH-1/4W" value="510"/>
-<part name="C26" library="rcl" deviceset="C-EU" device="C1206" value="0.1uF/250V"/>
+<part name="C26" library="SparkFun-Capacitors" deviceset="CAP" device="1210" value="1uF/100V"/>
 <part name="GND21" library="SparkFun-Aesthetics" deviceset="GND" device=""/>
 <part name="C27" library="rcl" deviceset="C-EU" device="C2220K" value="2.2uF/250V"/>
@@
 <part name="C4" library="SparkFun-Capacitors" deviceset="CAP_POL" device="PTH3" value="2200uF"/>
 <part name="C6" library="SparkFun-Capacitors" deviceset="1UF-25V-10%(0805)" device="&quot;" value="1uF"/>
-<part name="L1" library="SparkFun-Passives" deviceset="INDUCTOR" device="-B82462G" value="100u"/>
+<part name="L1" library="my" deviceset="INDUCTOR" device="NR10050T-PTH-ADD" value="220u"/>
 <part name="C2" library="SparkFun-Capacitors" deviceset="CAP_POL" device="PTH4" value="470uF"/>
 <part name="SUPPLY1" library="SparkFun-Aesthetics" deviceset="VCC" device=""/>
@@
 <part name="R14" library="SparkFun-Resistors" deviceset="100KOHM-1/10W-1%(0603)" device="" value="100k"/>
 <part name="R15" library="SparkFun-Resistors" deviceset="RESISTOR" device="PTH-1/2W" value="6.8/0.5W"/>
+<part name="R16" library="rcl" deviceset="R-US_" device="R0805" value="0.33"/>
 </parts>
 <sheets>
@@
 <instance part="R14" gate="G$1" x="119.38" y="203.2"/>
 <instance part="R15" gate="G$1" x="248.92" y="170.18"/>
+<instance part="R16" gate="G$1" x="43.18" y="187.96"/>
 </instances>
 <busses>
@@
 <pinref part="C26" gate="G$1" pin="2"/>
 <pinref part="GND21" gate="1" pin="GND"/>
+<wire x1="287.02" y1="121.92" x2="287.02" y2="124.46" width="0.1524" layer="91"/>
 </segment>
 <segment>
@@
 <wire x1="304.8" y1="132.08" x2="287.02" y2="132.08" width="0.1524" layer="91"/>
 <pinref part="C26" gate="G$1" pin="1"/>
-<wire x1="287.02" y1="132.08" x2="287.02" y2="129.54" width="0.1524" layer="91"/>
 </segment>
 </net>
@@
 <wire x1="76.2" y1="172.72" x2="76.2" y2="177.8" width="0.1524" layer="91"/>
 <label x="76.2" y="177.8" size="1.778" layer="95" rot="R90" xref="yes"/>
+<pinref part="R16" gate="G$1" pin="2"/>
+<wire x1="48.26" y1="187.96" x2="50.8" y2="187.96" width="0.1524" layer="91"/>
+<wire x1="50.8" y1="187.96" x2="50.8" y2="172.72" width="0.1524" layer="91"/>
+<junction x="50.8" y="172.72"/>
 </segment>
 <segment>
@@
 <wire x1="27.94" y1="157.48" x2="27.94" y2="172.72" width="0.1524" layer="91"/>
 <pinref part="L1" gate="G$1" pin="1"/>
-<wire x1="27.94" y1="172.72" x2="35.56" y2="172.72" width="0.1524" layer="91"/>
+<wire x1="27.94" y1="172.72" x2="33.02" y2="172.72" width="0.1524" layer="91"/>
+<wire x1="33.02" y1="172.72" x2="35.56" y2="172.72" width="0.1524" layer="91"/>
 <wire x1="27.94" y1="172.72" x2="25.4" y2="172.72" width="0.1524" layer="91"/>
 <junction x="27.94" y="172.72"/>
 <pinref part="SUPPLY1" gate="G$1" pin="VCC"/>
-</segment>
-<segment>
+<wire x1="33.02" y1="172.72" x2="33.02" y2="187.96" width="0.1524" layer="91"/>
+<junction x="33.02" y="172.72"/>
+<pinref part="R16" gate="G$1" pin="1"/>
+<wire x1="33.02" y1="187.96" x2="38.1" y2="187.96" width="0.1524" layer="91"/>
+</segment>
+<segment>

Commit message: HT filter added
Parts:
- added C28: 100uF/160V, SparkFun-Capacitors:CAP_POLPTH4
- added C29: 1uF/250V, rcl:C-EUC2220K
- added L2: 10u, SparkFun-Passives:INDUCTOR0805
- added R17: 0.33, SparkFun-Resistors:RESISTOR0805-RES
- C24: value 10uF/250V -> 10uF/160V; device SparkFun-Capacitors:CAP_POLG -> SparkFun-Capacitors:CAP_POLPTH4
Connections:
- new net N$7: C28.+, C29.1, L2.2, R17.2, U5.IN
- net GND: now also C28.-, C29.2
- net N$15: now also L2.1, R17.1; no longer U5.IN
Other:
- moved on the sheet: C24, C26, C27, R11, R12, R13, U5
Changed lines of the file:
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@@
 <part name="GND14" library="SparkFun-Aesthetics" deviceset="GND" device=""/>
 <part name="GND16" library="SparkFun-Aesthetics" deviceset="GND" device=""/>
-<part name="C24" library="SparkFun-Capacitors" deviceset="CAP_POL" device="G" value="10uF/250V"/>
+<part name="C24" library="SparkFun-Capacitors" deviceset="CAP_POL" device="PTH4" value="10uF/160V"/>
 <part name="GND19" library="SparkFun-Aesthetics" deviceset="GND" device=""/>
 <part name="U5" library="SparkFun-PowerIC" deviceset="V_REG_317" device="DPACK" value="LM317"/>
@@
 <part name="R15" library="SparkFun-Resistors" deviceset="RESISTOR" device="PTH-1/2W" value="6.8/0.5W"/>
 <part name="R16" library="rcl" deviceset="R-US_" device="R0805" value="0.33"/>
+<part name="L2" library="SparkFun-Passives" deviceset="INDUCTOR" device="0805" value="10u">
+<attribute name="MOUSER_PRICE" value="0.129"/>
+<attribute name="MOUSER_SKU" value="810-MLZ2012N100L"/>
+</part>
+<part name="R17" library="SparkFun-Resistors" deviceset="RESISTOR" device="0805-RES" value="0.33"/>
+<part name="C28" library="SparkFun-Capacitors" deviceset="CAP_POL" device="PTH4" value="100uF/160V"/>
+<part name="C29" library="rcl" deviceset="C-EU" device="C2220K" value="1uF/250V"/>
 </parts>
 <sheets>
@@
 <instance part="GND14" gate="1" x="223.52" y="88.9"/>
 <instance part="GND16" gate="1" x="254" y="88.9"/>
-<instance part="C24" gate="G$1" x="269.24" y="134.62"/>
-<instance part="GND19" gate="1" x="269.24" y="119.38"/>
-<instance part="U5" gate="G$1" x="304.8" y="144.78"/>
+<instance part="C24" gate="G$1" x="276.86" y="134.62"/>
+<instance part="GND19" gate="1" x="276.86" y="119.38"/>
+<instance part="U5" gate="G$1" x="335.28" y="144.78"/>
 <instance part="C25" gate="G$1" x="287.02" y="96.52"/>
 <instance part="GND20" gate="1" x="287.02" y="88.9"/>
-<instance part="R11" gate="G$1" x="304.8" y="127" rot="R90"/>
-<instance part="R13" gate="G$1" x="320.04" y="127" rot="R90"/>
-<instance part="GND22" gate="1" x="304.8" y="119.38"/>
-<instance part="R12" gate="G$1" x="320.04" y="139.7" rot="R90"/>
-<instance part="C26" gate="G$1" x="287.02" y="127"/>
-<instance part="GND21" gate="1" x="287.02" y="119.38"/>
-<instance part="C27" gate="G$1" x="332.74" y="137.16"/>
-<instance part="GND23" gate="1" x="332.74" y="119.38"/>
+<instance part="R11" gate="G$1" x="335.28" y="127" rot="R90"/>
+<instance part="R13" gate="G$1" x="350.52" y="127" rot="R90"/>
+<instance part="GND22" gate="1" x="335.28" y="119.38"/>
+<instance part="R12" gate="G$1" x="350.52" y="139.7" rot="R90"/>
+<instance part="C26" gate="G$1" x="317.5" y="127"/>
+<instance part="GND21" gate="1" x="317.5" y="119.38"/>
+<instance part="C27" gate="G$1" x="363.22" y="137.16"/>
+<instance part="GND23" gate="1" x="363.22" y="119.38"/>
 <instance part="IC1" gate="G$1" x="241.3" y="208.28"/>
 <instance part="GND15" gate="1" x="238.76" y="198.12"/>
@@
 <instance part="R15" gate="G$1" x="248.92" y="170.18"/>
 <instance part="R16" gate="G$1" x="43.18" y="187.96"/>
+<instance part="L2" gate="G$1" x="284.48" y="144.78" rot="R90">
+<attribute name="MOUSER_PRICE" x="284.48" y="144.78" size="1.778" layer="96" rot="R90" display="off"/>
+<attribute name="MOUSER_SKU" x="284.48" y="144.78" size="1.778" layer="96" rot="R90" display="off"/>
+</instance>
+<instance part="R17" gate="G$1" x="284.48" y="157.48"/>
+<instance part="C28" gate="G$1" x="292.1" y="134.62"/>
+<instance part="C29" gate="G$1" x="304.8" y="134.62"/>
 </instances>
 <busses>
@@
 <pinref part="C24" gate="G$1" pin="-"/>
 <pinref part="GND19" gate="1" pin="GND"/>
-<wire x1="269.24" y1="121.92" x2="269.24" y2="129.54" width="0.1524" layer="91"/>
+<wire x1="276.86" y1="121.92" x2="276.86" y2="127" width="0.1524" layer="91"/>
+<pinref part="C28" gate="G$1" pin="-"/>
+<wire x1="276.86" y1="127" x2="276.86" y2="129.54" width="0.1524" layer="91"/>
+<wire x1="292.1" y1="129.54" x2="292.1" y2="127" width="0.1524" layer="91"/>
+<wire x1="292.1" y1="127" x2="276.86" y2="127" width="0.1524" layer="91"/>
+<junction x="276.86" y="127"/>
+<pinref part="C29" gate="G$1" pin="2"/>
+<wire x1="304.8" y1="129.54" x2="304.8" y2="127" width="0.1524" layer="91"/>
+<wire x1="304.8" y1="127" x2="292.1" y2="127" width="0.1524" layer="91"/>
+<junction x="292.1" y="127"/>
 </segment>
 <segment>
@@
 <pinref part="R13" gate="G$1" pin="1"/>
 <pinref part="R11" gate="G$1" pin="1"/>
-<wire x1="320.04" y1="121.92" x2="304.8" y2="121.92" width="0.1524" layer="91"/>
+<wire x1="350.52" y1="121.92" x2="335.28" y2="121.92" width="0.1524" layer="91"/>
 <pinref part="GND22" gate="1" pin="GND"/>
-<junction x="304.8" y="121.92"/>
+<junction x="335.28" y="121.92"/>
 </segment>
 <segment>
 <pinref part="C26" gate="G$1" pin="2"/>
 <pinref part="GND21" gate="1" pin="GND"/>
-<wire x1="287.02" y1="121.92" x2="287.02" y2="124.46" width="0.1524" layer="91"/>
+<wire x1="317.5" y1="121.92" x2="317.5" y2="124.46" width="0.1524" layer="91"/>
 </segment>
 <segment>
 <pinref part="C27" gate="G$1" pin="2"/>
-<wire x1="332.74" y1="132.08" x2="332.74" y2="121.92" width="0.1524" layer="91"/>
+<wire x1="363.22" y1="132.08" x2="363.22" y2="121.92" width="0.1524" layer="91"/>
 <pinref part="GND23" gate="1" pin="GND"/>
 </segment>
@@
 <junction x="254" y="106.68"/>
 <wire x1="254" y1="106.68" x2="254" y2="144.78" width="0.1524" layer="91"/>
-<pinref part="U5" gate="G$1" pin="IN"/>
-<wire x1="254" y1="144.78" x2="269.24" y2="144.78" width="0.1524" layer="91"/>
+<wire x1="254" y1="144.78" x2="276.86" y2="144.78" width="0.1524" layer="91"/>
 <pinref part="C24" gate="G$1" pin="+"/>
-<wire x1="269.24" y1="144.78" x2="297.18" y2="144.78" width="0.1524" layer="91"/>
-<wire x1="269.24" y1="137.16" x2="269.24" y2="144.78" width="0.1524" layer="91"/>
-<junction x="269.24" y="144.78"/>
+<wire x1="276.86" y1="137.16" x2="276.86" y2="144.78" width="0.1524" layer="91"/>
+<junction x="276.86" y="144.78"/>
+<pinref part="L2" gate="G$1" pin="1"/>
+<pinref part="R17" gate="G$1" pin="1"/>
+<wire x1="279.4" y1="157.48" x2="276.86" y2="157.48" width="0.1524" layer="91"/>
+<wire x1="276.86" y1="157.48" x2="276.86" y2="144.78" width="0.1524" layer="91"/>
+<junction x="276.86" y="144.78"/>
 </segment>
 </net>
@@
 <pinref part="U5" gate="G$1" pin="ADJ"/>
 <pinref part="R11" gate="G$1" pin="2"/>
-<wire x1="304.8" y1="137.16" x2="304.8" y2="132.08" width="0.1524" layer="91"/>
+<wire x1="335.28" y1="137.16" x2="335.28" y2="132.08" width="0.1524" layer="91"/>
 <pinref part="R13" gate="G$1" pin="2"/>
-<wire x1="320.04" y1="132.08" x2="304.8" y2="132.08" width="0.1524" layer="91"/>
-<junction x="304.8" y="132.08"/>
+<wire x1="350.52" y1="132.08" x2="335.28" y2="132.08" width="0.1524" layer="91"/>
+<junction x="335.28" y="132.08"/>
 <pinref part="R12" gate="G$1" pin="1"/>
-<junction x="320.04" y="132.08"/>
-<wire x1="320.04" y1="132.08" x2="320.04" y2="134.62" width="0.1524" layer="91"/>
-<wire x1="304.8" y1="132.08" x2="287.02" y2="132.08" width="0.1524" layer="91"/>
+<junction x="350.52" y="132.08"/>
+<wire x1="350.52" y1="132.08" x2="350.52" y2="134.62" width="0.1524" layer="91"/>
+<wire x1="335.28" y1="132.08" x2="317.5" y2="132.08" width="0.1524" layer="91"/>
 <pinref part="C26" gate="G$1" pin="1"/>
 </segment>
@@
 <pinref part="U5" gate="G$1" pin="OUT"/>
 <pinref part="R12" gate="G$1" pin="2"/>
-<wire x1="312.42" y1="144.78" x2="320.04" y2="144.78" width="0.1524" layer="91"/>
-<wire x1="320.04" y1="144.78" x2="332.74" y2="144.78" width="0.1524" layer="91"/>
-<junction x="320.04" y="144.78"/>
+<wire x1="342.9" y1="144.78" x2="350.52" y2="144.78" width="0.1524" layer="91"/>
+<wire x1="350.52" y1="144.78" x2="363.22" y2="144.78" width="0.1524" layer="91"/>
+<junction x="350.52" y="144.78"/>
 <pinref part="C27" gate="G$1" pin="1"/>
-<wire x1="332.74" y1="144.78" x2="332.74" y2="139.7" width="0.1524" layer="91"/>
-<wire x1="332.74" y1="144.78" x2="337.82" y2="144.78" width="0.1524" layer="91"/>
-<junction x="332.74" y="144.78"/>
-<label x="337.82" y="144.78" size="1.778" layer="95" xref="yes"/>
+<wire x1="363.22" y1="144.78" x2="363.22" y2="139.7" width="0.1524" layer="91"/>
+<wire x1="363.22" y1="144.78" x2="368.3" y2="144.78" width="0.1524" layer="91"/>
+<junction x="363.22" y="144.78"/>
+<label x="368.3" y="144.78" size="1.778" layer="95" xref="yes"/>
 </segment>
 <segment>
@@
 </segment>
 </net>
+<net name="N$7" class="1">
+<segment>
+<pinref part="U5" gate="G$1" pin="IN"/>
+<wire x1="292.1" y1="144.78" x2="304.8" y2="144.78" width="0.1524" layer="91"/>
+<pinref part="L2" gate="G$1" pin="2"/>
+<pinref part="R17" gate="G$1" pin="2"/>
+<wire x1="304.8" y1="144.78" x2="327.66" y2="144.78" width="0.1524" layer="91"/>
+<wire x1="289.56" y1="157.48" x2="292.1" y2="157.48" width="0.1524" layer="91"/>
+<wire x1="292.1" y1="157.48" x2="292.1" y2="144.78" width="0.1524" layer="91"/>
+<junction x="292.1" y="144.78"/>
+<pinref part="C28" gate="G$1" pin="+"/>
+<wire x1="292.1" y1="137.16" x2="292.1" y2="144.78" width="0.1524" layer="91"/>
+<pinref part="C29" gate="G$1" pin="1"/>
+<wire x1="304.8" y1="137.16" x2="304.8" y2="144.78" width="0.1524" layer="91"/>
+<junction x="304.8" y="144.78"/>
+</segment>
+</net>

Commit message: Unneeded resistors
Parts:
- removed R16: 0.33, rcl:R-US_R0805
- removed R17: 0.33, SparkFun-Resistors:RESISTOR0805-RES
- L2: value 10u -> 100u; device SparkFun-Passives:INDUCTOR0805 -> SparkFun-Passives:INDUCTOR1210; MOUSER_PRICE 0.129 -> 0.168; MOUSER_SKU 810-MLZ2012N100L -> 963-LB3218T101K
Connections:
- net N$15: no longer R17.1
- net N$7: no longer R17.2
- net VCC: no longer R16.1
- net VINF: no longer R16.2
Changed lines of the file:
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@@
 <part name="R14" library="SparkFun-Resistors" deviceset="100KOHM-1/10W-1%(0603)" device="" value="100k"/>
 <part name="R15" library="SparkFun-Resistors" deviceset="RESISTOR" device="PTH-1/2W" value="6.8/0.5W"/>
-<part name="R16" library="rcl" deviceset="R-US_" device="R0805" value="0.33"/>
-<part name="L2" library="SparkFun-Passives" deviceset="INDUCTOR" device="0805" value="10u">
-<attribute name="MOUSER_PRICE" value="0.129"/>
-<attribute name="MOUSER_SKU" value="810-MLZ2012N100L"/>
+<part name="L2" library="SparkFun-Passives" deviceset="INDUCTOR" device="1210" value="100u">
+<attribute name="MOUSER_PRICE" value="0.168"/>
+<attribute name="MOUSER_SKU" value="963-LB3218T101K"/>
 </part>
-<part name="R17" library="SparkFun-Resistors" deviceset="RESISTOR" device="0805-RES" value="0.33"/>
 <part name="C28" library="SparkFun-Capacitors" deviceset="CAP_POL" device="PTH4" value="100uF/160V"/>
 <part name="C29" library="rcl" deviceset="C-EU" device="C2220K" value="1uF/250V"/>
@@
 <instance part="R14" gate="G$1" x="119.38" y="203.2"/>
 <instance part="R15" gate="G$1" x="248.92" y="170.18"/>
-<instance part="R16" gate="G$1" x="43.18" y="187.96"/>
 <instance part="L2" gate="G$1" x="284.48" y="144.78" rot="R90">
 <attribute name="MOUSER_PRICE" x="284.48" y="144.78" size="1.778" layer="96" rot="R90" display="off"/>
 <attribute name="MOUSER_SKU" x="284.48" y="144.78" size="1.778" layer="96" rot="R90" display="off"/>
 </instance>
-<instance part="R17" gate="G$1" x="284.48" y="157.48"/>
 <instance part="C28" gate="G$1" x="292.1" y="134.62"/>
 <instance part="C29" gate="G$1" x="304.8" y="134.62"/>
@@
 <junction x="276.86" y="144.78"/>
 <pinref part="L2" gate="G$1" pin="1"/>
-<pinref part="R17" gate="G$1" pin="1"/>
-<wire x1="279.4" y1="157.48" x2="276.86" y2="157.48" width="0.1524" layer="91"/>
-<wire x1="276.86" y1="157.48" x2="276.86" y2="144.78" width="0.1524" layer="91"/>
 <junction x="276.86" y="144.78"/>
 </segment>
@@
 <wire x1="76.2" y1="172.72" x2="76.2" y2="177.8" width="0.1524" layer="91"/>
 <label x="76.2" y="177.8" size="1.778" layer="95" rot="R90" xref="yes"/>
-<pinref part="R16" gate="G$1" pin="2"/>
-<wire x1="48.26" y1="187.96" x2="50.8" y2="187.96" width="0.1524" layer="91"/>
-<wire x1="50.8" y1="187.96" x2="50.8" y2="172.72" width="0.1524" layer="91"/>
-<junction x="50.8" y="172.72"/>
 </segment>
 <segment>
@@
 <wire x1="27.94" y1="157.48" x2="27.94" y2="172.72" width="0.1524" layer="91"/>
 <pinref part="L1" gate="G$1" pin="1"/>
-<wire x1="27.94" y1="172.72" x2="33.02" y2="172.72" width="0.1524" layer="91"/>
-<wire x1="33.02" y1="172.72" x2="35.56" y2="172.72" width="0.1524" layer="91"/>
+<wire x1="27.94" y1="172.72" x2="35.56" y2="172.72" width="0.1524" layer="91"/>
 <wire x1="27.94" y1="172.72" x2="25.4" y2="172.72" width="0.1524" layer="91"/>
 <junction x="27.94" y="172.72"/>
 <pinref part="SUPPLY1" gate="G$1" pin="VCC"/>
-<wire x1="33.02" y1="172.72" x2="33.02" y2="187.96" width="0.1524" layer="91"/>
-<junction x="33.02" y="172.72"/>
-<pinref part="R16" gate="G$1" pin="1"/>
-<wire x1="33.02" y1="187.96" x2="38.1" y2="187.96" width="0.1524" layer="91"/>
 </segment>
 <segment>
@@
 <wire x1="292.1" y1="144.78" x2="304.8" y2="144.78" width="0.1524" layer="91"/>
 <pinref part="L2" gate="G$1" pin="2"/>
-<pinref part="R17" gate="G$1" pin="2"/>
 <wire x1="304.8" y1="144.78" x2="327.66" y2="144.78" width="0.1524" layer="91"/>
-<wire x1="289.56" y1="157.48" x2="292.1" y2="157.48" width="0.1524" layer="91"/>
-<wire x1="292.1" y1="157.48" x2="292.1" y2="144.78" width="0.1524" layer="91"/>
 <junction x="292.1" y="144.78"/>
 <pinref part="C28" gate="G$1" pin="+"/>
