File: ps2/ps2.sch (EAGLE design)
At the start: 47 parts, among them U1 LM317, U2 LM317, U3 LM317, U4 LM337

Commit message: Small tweak
Parts:
- C2: device rcl:CPOL-USE3.5-8 -> SparkFun-Capacitors:CAP_POLPTH1
Changed lines of the file:
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@@
 <part name="C10" library="rcl" deviceset="C-EU" device="C1206" value="1uF/100V"/>
 <part name="GND3" library="SparkFun-Aesthetics" deviceset="GND" device=""/>
-<part name="C2" library="rcl" deviceset="CPOL-US" device="E3.5-8" value="10uF/100V"/>
+<part name="C2" library="SparkFun-Capacitors" deviceset="CAP_POL" device="PTH1" value="10uF/100V"/>
 <part name="U2" library="SparkFun-PowerIC" deviceset="V_REG_317" device="DPACK" value="LM317"/>
 <part name="R3" library="SparkFun-Resistors" deviceset="RESISTOR" device="PTH-1/4W" value="240"/>
