File: ps2/ps2.brd (EAGLE design)
At the start: 99.1 x 74.9 mm, 47 parts, among them U1 LM317, U2 LM317, U3 LM317, U4 LM337

Commit message: Small tweak
Parts:
- C2: device rcl:E3,5-8 -> SparkFun-Capacitors:CPOL-RADIAL-100UF-25V
- moved C2 1.27 mm to (55.9, 52.1), turned to 90 degrees
Connections:
- net GND: now also C2.2; no longer C2.-
- net N$5: now also C2.1; no longer C2.+
Changed lines of the file:
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@@
 <attribute name="VALUE" x="89.535" y="41.91" size="0.8128" layer="27" ratio="15" rot="R180"/>
 </element>
-<element name="C2" library="rcl" package="E3,5-8" value="10uF/100V" x="54.61" y="52.07" smashed="yes" rot="R270">
-<attribute name="NAME" x="52.197" y="53.594" size="0.8128" layer="25" ratio="15"/>
-<attribute name="VALUE" x="59.182" y="55.626" size="0.8128" layer="27" ratio="15" rot="R270"/>
+<element name="C2" library="SparkFun-Capacitors" package="CPOL-RADIAL-100UF-25V" value="10uF/100V" x="55.88" y="52.07" smashed="yes" rot="R90">
+<attribute name="NAME" x="58.293" y="50.546" size="0.8128" layer="25" ratio="15" rot="R180"/>
+<attribute name="VALUE" x="51.308" y="48.514" size="0.8128" layer="27" ratio="15" rot="R90"/>
 </element>
 <element name="U2" library="SparkFun-PowerIC" package="V-REG_DPACK" value="LM317" x="81.28" y="66.04" smashed="yes" rot="R270">
@@
 <contactref element="C9" pad="-"/>
 <contactref element="C10" pad="2"/>
-<contactref element="C2" pad="-"/>
+<contactref element="C2" pad="2"/>
 <contactref element="R4" pad="P$1"/>
 <contactref element="C11" pad="2"/>
@@
 <contactref element="U1" pad="1"/>
 <contactref element="D9" pad="A"/>
-<contactref element="C2" pad="+"/>
-<wire x1="54.61" y1="53.848" x2="55.112" y2="54.35" width="2.54" layer="1" curve="-90"/>
-<wire x1="55.112" y1="54.35" x2="58.42" y2="54.35" width="2.54" layer="1"/>
+<contactref element="C2" pad="1"/>
 <wire x1="58.42" y1="54.35" x2="62.51" y2="54.35" width="2.54" layer="1"/>
-<wire x1="52.07" y1="58.42" x2="54.61" y2="55.88" width="2.54" layer="1" curve="-90"/>
-<wire x1="54.61" y1="55.88" x2="54.61" y2="53.848" width="2.54" layer="1"/>
 <wire x1="62.23" y1="62.23" x2="58.42" y2="58.42" width="2.54" layer="1" curve="90"/>
 <wire x1="58.42" y1="58.42" x2="58.42" y2="54.35" width="2.54" layer="1"/>
 <wire x1="62.23" y1="62.23" x2="65.16" y2="62.23" width="2.54" layer="1"/>
 <wire x1="65.16" y1="62.23" x2="66.04" y2="63.11" width="2.54" layer="1" curve="90"/>
+<wire x1="58.42" y1="54.35" x2="56.14" y2="54.35" width="2.54" layer="1"/>
+<wire x1="56.14" y1="54.35" x2="52.07" y2="58.42" width="2.54" layer="1" curve="-90"/>
+<wire x1="55.88" y1="53.34" x2="55.88" y2="54.09" width="2.54" layer="1"/>
+<wire x1="55.88" y1="54.09" x2="56.14" y2="54.35" width="2.54" layer="1" curve="-90"/>
 </signal>
 <signal name="+60V">

Commit message: Small tweak
Parts:
- moved D4 17.2 mm to (26.0, 55.2), turned to 0 degrees
- moved D3 3.24 mm to (33.7, 55.2)
- moved D8 2.62 mm to (40.6, 55.2)
Routing:
- net N$1: track 32.3 -> 14.5 mm
- net LS: track 66.6 -> 64.2 mm
- net +HV: track 31.1 -> 29.4 mm
Changed lines of the file:
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@@
 <attribute name="NAME" x="25.4" y="69.85" size="0.8128" layer="25" ratio="15"/>
 </element>
-<element name="D4" library="SparkFun-DiscreteSemi" package="SMA-DIODE" value="2A" x="12.7" y="66.04" smashed="yes" rot="R180">
-<attribute name="NAME" x="14.986" y="64.389" size="0.8128" layer="25" ratio="15" rot="R180"/>
-<attribute name="VALUE" x="12.446" y="64.389" size="0.8128" layer="27" ratio="15" rot="R180"/>
+<element name="D4" library="SparkFun-DiscreteSemi" package="SMA-DIODE" value="2A" x="26.035" y="55.245" smashed="yes">
+<attribute name="NAME" x="23.749" y="56.896" size="0.8128" layer="25" ratio="15"/>
+<attribute name="VALUE" x="26.289" y="56.896" size="0.8128" layer="27" ratio="15"/>
 </element>
 <element name="C3" library="SparkFun-Capacitors" package="CPOL-RADIAL-1000UF-63V" value="470uF/100V" x="25.4" y="44.45" smashed="yes">
@@
 <attribute name="NAME" x="24.765" y="48.26" size="0.8128" layer="25" ratio="15"/>
 </element>
-<element name="D3" library="SparkFun-DiscreteSemi" package="SMA-DIODE" value="2A" x="30.48" y="55.88" smashed="yes">
-<attribute name="NAME" x="28.194" y="57.531" size="0.8128" layer="25" ratio="15"/>
-<attribute name="VALUE" x="30.734" y="57.531" size="0.8128" layer="27" ratio="15"/>
+<element name="D3" library="SparkFun-DiscreteSemi" package="SMA-DIODE" value="2A" x="33.655" y="55.245" smashed="yes">
+<attribute name="NAME" x="31.369" y="56.896" size="0.8128" layer="25" ratio="15"/>
+<attribute name="VALUE" x="33.909" y="56.896" size="0.8128" layer="27" ratio="15"/>
 </element>
 <element name="C4" library="SparkFun-Capacitors" package="CPOL-RADIAL-1000UF-63V" value="470uF/100V" x="43.18" y="44.45" smashed="yes" rot="R90">
@@
 <attribute name="NAME" x="42.545" y="50.165" size="0.8128" layer="25" ratio="15"/>
 </element>
-<element name="D8" library="SparkFun-DiscreteSemi" package="SMA-DIODE" value="2A" x="38.1" y="55.88" smashed="yes">
-<attribute name="NAME" x="35.814" y="57.531" size="0.8128" layer="25" ratio="15"/>
-<attribute name="VALUE" x="38.354" y="57.531" size="0.8128" layer="27" ratio="15"/>
+<element name="D8" library="SparkFun-DiscreteSemi" package="SMA-DIODE" value="2A" x="40.64" y="55.245" smashed="yes">
+<attribute name="NAME" x="38.354" y="56.896" size="0.8128" layer="25" ratio="15"/>
+<attribute name="VALUE" x="40.894" y="56.896" size="0.8128" layer="27" ratio="15"/>
 </element>
 <element name="U3" library="SparkFun-PowerIC" package="V-REG_DPACK" value="LM317" x="67.31" y="11.43" smashed="yes" rot="R270">
@@
 <via x="25.4" y="46.99" extent="1-16" drill="0.6"/>
 <via x="25.4" y="50.8" extent="1-16" drill="0.6"/>
-<via x="25.4" y="54.61" extent="1-16" drill="0.6"/>
 <via x="24.13" y="58.42" extent="1-16" drill="0.6"/>
-<via x="17.78" y="62.23" extent="1-16" drill="0.6"/>
+<via x="16.51" y="62.865" extent="1-16" drill="0.6"/>
 <via x="20.32" y="63.5" extent="1-16" drill="0.6"/>
 <via x="24.13" y="64.77" extent="1-16" drill="0.6"/>
 <via x="25.4" y="67.31" extent="1-16" drill="0.6"/>
 <via x="28.575" y="47.625" extent="1-16" drill="0.6"/>
-<via x="29.845" y="51.435" extent="1-16" drill="0.6"/>
-<via x="35.56" y="52.07" extent="1-16" drill="0.6"/>
-<via x="35.56" y="48.26" extent="1-16" drill="0.6"/>
-<via x="34.29" y="44.45" extent="1-16" drill="0.6"/>
+<via x="32.385" y="50.165" extent="1-16" drill="0.6"/>
+<via x="38.1" y="45.72" extent="1-16" drill="0.6"/>
+<via x="35.56" y="43.18" extent="1-16" drill="0.6"/>
 <via x="31.75" y="41.91" extent="1-16" drill="0.6"/>
 <via x="27.94" y="41.91" extent="1-16" drill="0.6"/>
 <via x="39.37" y="52.07" extent="1-16" drill="0.6"/>
 <via x="39.37" y="48.26" extent="1-16" drill="0.6"/>
-<via x="40.64" y="44.45" extent="1-16" drill="0.6"/>
+<via x="41.91" y="43.18" extent="1-16" drill="0.6"/>
 <via x="45.72" y="41.91" extent="1-16" drill="0.6"/>
 <via x="49.53" y="41.91" extent="1-16" drill="0.6"/>
@@
 <via x="39.37" y="59.055" extent="1-16" drill="0.6"/>
 <via x="43.18" y="59.055" extent="1-16" drill="0.6"/>
-<via x="45.72" y="57.15" extent="1-16" drill="0.6"/>
 <via x="46.99" y="54.61" extent="1-16" drill="0.6"/>
 <via x="46.99" y="50.8" extent="1-16" drill="0.6"/>
 <via x="49.53" y="49.53" extent="1-16" drill="0.6"/>
 <via x="52.07" y="52.07" extent="1-16" drill="0.6"/>
-<via x="50.8" y="55.88" extent="1-16" drill="0.6"/>
 <via x="49.53" y="59.69" extent="1-16" drill="0.6"/>
 <via x="49.53" y="63.5" extent="1-16" drill="0.6"/>
@@
 <wire x1="4.445" y1="27.695" x2="10.55" y2="21.59" width="2.54" layer="1" curve="90"/>
 <wire x1="10.55" y1="15.24" x2="10.55" y2="21.59" width="2.54" layer="1"/>
-<wire x1="21.59" y1="44.45" x2="21.59" y2="52.95" width="2.54" layer="1"/>
-<wire x1="21.59" y1="52.95" x2="14.85" y2="59.69" width="2.54" layer="1" curve="90"/>
-<wire x1="14.85" y1="59.69" x2="14.85" y2="66.04" width="2.54" layer="1"/>
+<wire x1="21.59" y1="44.45" x2="21.59" y2="55.245" width="2.54" layer="1"/>
+<wire x1="21.59" y1="55.245" x2="21.59" y2="55.88" width="2.54" layer="1"/>
 <wire x1="4.445" y1="33.02" x2="5.715" y2="34.29" width="2.54" layer="1" curve="-90"/>
 <wire x1="5.715" y1="34.29" x2="11.43" y2="34.29" width="2.54" layer="1"/>
 <wire x1="11.43" y1="34.29" x2="21.59" y2="44.45" width="2.54" layer="1" curve="90"/>
+<wire x1="21.59" y1="55.88" x2="17.78" y2="59.69" width="2.54" layer="1" curve="90"/>
+<wire x1="17.78" y1="59.69" x2="14.85" y2="59.69" width="2.54" layer="1"/>
+<wire x1="23.885" y1="55.245" x2="21.59" y2="55.245" width="2.54" layer="1"/>
 </signal>
 <signal name="HS">
@@
 <contactref element="D3" pad="A"/>
 <contactref element="D4" pad="C"/>
-<wire x1="28.33" y1="55.88" x2="28.33" y2="65.16" width="2.54" layer="1"/>
-<wire x1="28.33" y1="65.16" x2="29.21" y2="66.04" width="2.54" layer="1" curve="-90"/>
-<wire x1="10.55" y1="66.04" x2="14.36" y2="69.85" width="2.54" layer="1" curve="-90"/>
-<wire x1="14.36" y1="69.85" x2="25.4" y2="69.85" width="2.54" layer="1"/>
-<wire x1="25.4" y1="69.85" x2="29.21" y2="66.04" width="2.54" layer="1" curve="-90"/>
+<wire x1="28.185" y1="55.245" x2="31.505" y2="55.245" width="2.54" layer="1"/>
+<wire x1="28.185" y1="55.245" x2="29.21" y2="56.27" width="2.54" layer="1" curve="90"/>
+<wire x1="29.21" y1="56.27" x2="29.21" y2="66.04" width="2.54" layer="1"/>
 </signal>
 <signal name="N$2">
@@
 <contactref element="C3" pad="1"/>
 <contactref element="D8" pad="A"/>
-<wire x1="29.21" y1="44.45" x2="32.63" y2="47.87" width="2.54" layer="1" curve="90"/>
-<wire x1="32.63" y1="47.87" x2="32.63" y2="55.88" width="2.54" layer="1"/>
-<wire x1="32.63" y1="55.88" x2="35.95" y2="55.88" width="2.54" layer="1"/>
+<wire x1="35.805" y1="55.245" x2="38.49" y2="55.245" width="2.54" layer="1"/>
+<wire x1="29.21" y1="44.45" x2="35.805" y2="51.045" width="2.54" layer="1" curve="90"/>
+<wire x1="35.805" y1="51.045" x2="35.805" y2="55.245" width="2.54" layer="1"/>
 </signal>
 <signal name="+HV">
@@
 <contactref element="D5" pad="C"/>
 <contactref element="U1" pad="3"/>
-<wire x1="40.25" y1="55.88" x2="43.18" y2="52.95" width="2.54" layer="1" curve="-90"/>
-<wire x1="43.18" y1="52.95" x2="43.18" y2="48.26" width="2.54" layer="1"/>
 <wire x1="43.18" y1="48.26" x2="45.72" y2="45.72" width="2.54" layer="1" curve="90"/>
 <wire x1="45.72" y1="45.72" x2="58.81" y2="45.72" width="2.54" layer="1"/>
 <wire x1="58.81" y1="45.72" x2="58.81" y2="46.09" width="2.54" layer="1"/>
 <wire x1="58.81" y1="46.09" x2="62.51" y2="49.79" width="2.54" layer="1" curve="-90"/>
+<wire x1="43.18" y1="48.26" x2="43.18" y2="54.855" width="2.54" layer="1"/>
+<wire x1="43.18" y1="54.855" x2="42.79" y2="55.245" width="2.54" layer="1" curve="90"/>
 </signal>
 <signal name="+12V">
